Commit message: Add LiDAR and Twist_MUX

File: src/bumperbot_description/urdf/bumperbot.urdf.xacro (robot description, xacro)
@@ -166,3 +166,30 @@
     <child link="imu_link" />
   </joint>
+    <link name="laser_link">
+    <inertial>
+      <origin xyz="-0.011945780406062 -0.000381929217680526 -0.0170649378129477" rpy="0 0 0" />
+      <mass value="0.073084435549317" />
+      <inertia ixx="1.96074931730795E-05" ixy="-3.62091076640009E-07" ixz="4.28230084046735E-07"
+               iyy="2.40983835136327E-05" iyz="1.50180909250652E-08"
+               izz="4.14184164228595E-05" />
+    </inertial>
+    <visual>
+      <origin xyz="0 0 0" rpy="0 0 0" />
+      <geometry>
+        <mesh filename="package://bumperbot_description/meshes/laser_link.STL" />
+      </geometry>
+    </visual>
+    <collision>
+      <origin xyz="0 0 0" rpy="0 0 0" />
+      <geometry>
+        <mesh filename="package://bumperbot_description/meshes/laser_link.STL" />
+      </geometry>
+    </collision>
+  </link>
+  <joint name="laser_joint" type="fixed">
+    <origin xyz="-0.0050526 -0.0023221 0.1208" rpy="0 0 3.14" />
+    <parent link="base_link" />
+    <child link="laser_link" />
+    <axis xyz="0 0 0" />
+  </joint>
 </robot>

File: src/bumperbot_description/urdf/bumperbot_gazebo.xacro (robot description, xacro)
@@ -43,7 +43,7 @@
         <plugin filename="gz-sim-imu-system" name="gz::sim::systems::Imu"/>
         <!-- Camera / LiDAR -->
-        <!-- <plugin filename="gz-sim-sensors-system" name="gz::sim::systems::Sensors">
+        <plugin filename="gz-sim-sensors-system" name="gz::sim::systems::Sensors">
             <render_engine>ogre2</render_engine>
-        </plugin> -->
+        </plugin>
     </gazebo>
     <!-- IMU -->
@@ -98,3 +98,33 @@
         </sensor>
     </gazebo>
+    <!-- 2D Laser Sensor -->
+    <gazebo reference="laser_link">
+        <sensor name="lidar" type="gpu_lidar">
+        <always_on>true</always_on>
+        <visualize>true</visualize>
+        <topic>scan</topic>
+        <update_rate>5</update_rate>
+        <gz_frame_id>laser_link</gz_frame_id>
+        <lidar>
+            <scan>
+                <horizontal>
+                    <samples>360</samples>
+                    <resolution>1.00000</resolution>
+                    <min_angle>0.000000</min_angle>
+                    <max_angle>6.280000</max_angle>
+                </horizontal>
+            </scan>
+            <range>
+                <min>0.120000</min>
+                <max>12.0</max>
+                <resolution>0.02</resolution>
+            </range>
+            <noise>
+                <type>gaussian</type>
+                <mean>0.0</mean>
+                <stddev>0.01</stddev>
+            </noise>
+        </lidar>
+        </sensor>
+    </gazebo>
 </robot>
